Commit message: sfg_peripherals_description: Work on luxonis_oakd_pro.xacro.

File: sfg_peripherals_description/xacro/luxonis_oakd_pro.xacro (robot description, xacro)
@@ -16,5 +16,43 @@
             </visual>
         </link>
-        <!-- ToDo Implement frames for different camera streams. -->
+        <!-- color -->
+        <joint name="${name}_color_frame_joint" type="fixed">
+            <parent link="${name}" />
+            <child link="${name}_color_frame" />
+            <origin rpy="0 0 0" xyz="0 0 0.02" />
+        </joint>
+        <link name="${name}_color_frame" />
+        <joint name="${name}_color_optical_frame_joint" type="fixed">
+            <parent link="${name}_color_frame" />
+            <child link="${name}_color_optical_frame" />
+            <origin rpy="${-0.5 * pi} 0 ${-0.5 * pi}" xyz="0 0 0" />
+        </joint>
+        <link name="${name}_color_optical_frame" />
+        <!-- mono left -->
+        <joint name="${name}_mono_left_frame_joint" type="fixed">
+            <parent link="${name}" />
+            <child link="${name}_mono_left_frame" />
+            <origin rpy="0 0 0" xyz="0.0375 0 0.02" />
+        </joint>
+        <link name="${name}_mono_left_frame" />
+        <joint name="${name}_mono_left_optical_frame_joint" type="fixed">
+            <parent link="${name}_mono_left_frame" />
+            <child link="${name}_mono_left_optical_frame" />
+            <origin rpy="${-0.5 * pi} 0 ${-0.5 * pi}" xyz="0 0 0" />
+        </joint>
+        <link name="${name}_mono_left_optical_frame" />
+        <!-- mono right -->
+        <joint name="${name}_mono_right_frame_joint" type="fixed">
+            <parent link="${name}" />
+            <child link="${name}_mono_right_frame" />
+            <origin rpy="0 0 0" xyz="-0.0375 0 0.02" />
+        </joint>
+        <link name="${name}_mono_right_frame" />
+        <joint name="${name}_mono_right_optical_frame_joint" type="fixed">
+            <parent link="${name}_mono_right_frame" />
+            <child link="${name}_mono_right_optical_frame" />
+            <origin rpy="${-0.5 * pi} 0 ${-0.5 * pi}" xyz="0 0 0" />
+        </joint>
+        <link name="${name}_mono_right_optical_frame" />
     </xacro:macro>
 </robot>

Commit message: sfg_peripherals_description: Updated oakd_pro xacro.

File: sfg_peripherals_description/xacro/luxonis_oakd_pro.xacro (robot description, xacro)
@@ -16,9 +16,15 @@
             </visual>
         </link>
+        <joint name="${name}_base_frame_joint" type="fixed">
+            <parent link="${name}" />
+            <child link="${name}_base_frame" />
+            <origin rpy="0 0 0" xyz="0 0.00476 0.02273" />
+        </joint>
+        <link name="${name}_base_frame" />
         <!-- color -->
         <joint name="${name}_color_frame_joint" type="fixed">
-            <parent link="${name}" />
+            <parent link="${name}_base_frame" />
             <child link="${name}_color_frame" />
-            <origin rpy="0 0 0" xyz="0 0 0.02" />
+            <origin rpy="0 0 0" xyz="0 0 0" />
         </joint>
         <link name="${name}_color_frame" />
@@ -31,7 +37,7 @@
         <!-- mono left -->
         <joint name="${name}_mono_left_frame_joint" type="fixed">
-            <parent link="${name}" />
+            <parent link="${name}_base_frame" />
             <child link="${name}_mono_left_frame" />
-            <origin rpy="0 0 0" xyz="0.0375 0 0.02" />
+            <origin rpy="0 0 0" xyz="0.0375 0 0" />
         </joint>
         <link name="${name}_mono_left_frame" />
@@ -44,7 +50,7 @@
         <!-- mono right -->
         <joint name="${name}_mono_right_frame_joint" type="fixed">
-            <parent link="${name}" />
+            <parent link="${name}_base_frame" />
             <child link="${name}_mono_right_frame" />
-            <origin rpy="0 0 0" xyz="-0.0375 0 0.02" />
+            <origin rpy="0 0 0" xyz="-0.0375 0 0" />
         </joint>
         <link name="${name}_mono_right_frame" />
