Commit message: sfg_peripherals_description: Ensured all collada meshes are oriented in a consistent manner and fixed coordinate frames for OAK-D.

File: sfg_peripherals_description/xacro/livox_mid360.xacro (robot description, xacro)
@@ -18,5 +18,5 @@
             <parent link="${name}" />
             <child link="${name}_point_cloud_frame" />
-            <origin rpy="0 0 0" xyz="0 0 0.047" />
+            <origin rpy="0 0 ${pi}" xyz="0 0 0.047" />
         </joint>
         <link name="${name}_point_cloud_frame" />
@@ -24,5 +24,5 @@
             <parent link="${name}" />
             <child link="${name}_imu_frame" />
-            <origin rpy="0 0 0" xyz="-0.02329 -0.011 0.00288" />
+            <origin rpy="0 0 ${pi}" xyz="-0.02329 -0.011 0.00288" />
         </joint>
         <link name="${name}_imu_frame" />

File: sfg_peripherals_description/xacro/luxonis_oakd_pro.xacro (robot description, xacro)
@@ -19,5 +19,5 @@
             <parent link="${name}" />
             <child link="${name}_base_frame" />
-            <origin rpy="0 0 0" xyz="0 0.00476 0.02273" />
+            <origin rpy="0 ${-0.5 * pi} 0" xyz="0 0.00476 0.02273" />
         </joint>
         <link name="${name}_base_frame" />
@@ -39,5 +39,5 @@
             <parent link="${name}_base_frame" />
             <child link="${name}_mono_left_frame" />
-            <origin rpy="0 0 0" xyz="0.0375 0 0" />
+            <origin rpy="0 0 0" xyz="0 0.0375 0" />
         </joint>
         <link name="${name}_mono_left_frame" />
@@ -52,5 +52,5 @@
             <parent link="${name}_base_frame" />
             <child link="${name}_mono_right_frame" />
-            <origin rpy="0 0 0" xyz="-0.0375 0 0" />
+            <origin rpy="0 0 0" xyz="0 -0.0375 0" />
         </joint>
         <link name="${name}_mono_right_frame" />
