Commit message: Fixed wrong filepath to mesh in htc_vive_tracker_30.xacro.

File: sfg_peripherals_description/xacro/htc_vive_tracker_30.xacro (robot description, xacro)
@@ -10,5 +10,7 @@
             <visual>
                 <geometry>
-                    <mesh filename="package://sfg_go2_description/mesh/tracker.dae" scale="1 1 1" />
+                    <mesh
+                        filename="package://sfg_peripherals_description/mesh/htc_vive_tracker_30.dae"
+                        scale="1 1 1" />
                 </geometry>
             </visual>

Commit message: Fixed wrong indent size for xacro/xml files.

File: sfg_peripherals_description/xacro/htc_vive_tracker_30.xacro (robot description, xacro)
@@ -1,25 +1,25 @@
 <?xml version="1.0"?>
 <robot xmlns:xacro="http://www.ros.org/wiki/xacro">
-    <xacro:macro name="htc_vive_tracker_30" params="name parent *origin">
-        <joint name="${name}_joint" type="fixed">
-            <parent link="${parent}" />
-            <child link="${name}" />
-            <xacro:insert_block name="origin" />
-        </joint>
-        <link name="${name}">
-            <visual>
-                <geometry>
-                    <mesh
-                        filename="package://sfg_peripherals_description/mesh/htc_vive_tracker_30.dae"
-                        scale="1 1 1" />
-                </geometry>
-            </visual>
-        </link>
-        <joint name="${name}_frame_joint" type="fixed">
-            <parent link="${name}" />
-            <child link="${name}_frame" />
-            <origin rpy="${0.5 * pi} 0 ${-0.5 * pi}" xyz="0 0 0.0005" />
-        </joint>
-        <link name="${name}_frame" />
-    </xacro:macro>
+  <xacro:macro name="htc_vive_tracker_30" params="name parent *origin">
+    <joint name="${name}_joint" type="fixed">
+      <parent link="${parent}" />
+      <child link="${name}" />
+      <xacro:insert_block name="origin" />
+    </joint>
+    <link name="${name}">
+      <visual>
+        <geometry>
+          <mesh
+            filename="package://sfg_peripherals_description/mesh/htc_vive_tracker_30.dae"
+            scale="1 1 1" />
+        </geometry>
+      </visual>
+    </link>
+    <joint name="${name}_frame_joint" type="fixed">
+      <parent link="${name}" />
+      <child link="${name}_frame" />
+      <origin rpy="${0.5 * pi} 0 ${-0.5 * pi}" xyz="0 0 0.0005" />
+    </joint>
+    <link name="${name}_frame" />
+  </xacro:macro>
 </robot>

File: sfg_peripherals_description/xacro/intel_realsense_d435.xacro (robot description, xacro)
@@ -1,25 +1,25 @@
 <?xml version="1.0"?>
 <robot xmlns:xacro="http://www.ros.org/wiki/xacro">
-    <xacro:macro name="intel_realsense_d435" params="name parent *origin">
-        <joint name="${name}_joint" type="fixed">
-            <parent link="${parent}" />
-            <child link="${name}" />
-            <xacro:insert_block name="origin" />
-        </joint>
-        <link name="${name}">
-            <visual>
-                <geometry>
-                    <mesh
-                        filename="package://sfg_peripherals_description/mesh/intel_realsense_d435.dae"
-                        scale="1 1 1" />
-                </geometry>
-            </visual>
-        </link>
-        <joint name="${name}_base_frame_joint" type="fixed">
-            <parent link="${name}" />
-            <child link="${name}_base_frame" />
-            <origin rpy="0 ${-0.5 * pi} 0" xyz="0 0.0175 0.02075" />
-        </joint>
-        <link name="${name}_base_frame" />
-    </xacro:macro>
+  <xacro:macro name="intel_realsense_d435" params="name parent *origin">
+    <joint name="${name}_joint" type="fixed">
+      <parent link="${parent}" />
+      <child link="${name}" />
+      <xacro:insert_block name="origin" />
+    </joint>
+    <link name="${name}">
+      <visual>
+        <geometry>
+          <mesh
+            filename="package://sfg_peripherals_description/mesh/intel_realsense_d435.dae"
+            scale="1 1 1" />
+        </geometry>
+      </visual>
+    </link>
+    <joint name="${name}_base_frame_joint" type="fixed">
+      <parent link="${name}" />
+      <child link="${name}_base_frame" />
+      <origin rpy="0 ${-0.5 * pi} 0" xyz="0 0.0175 0.02075" />
+    </joint>
+    <link name="${name}_base_frame" />
+  </xacro:macro>
 </robot>

File: sfg_peripherals_description/xacro/livox_mid360.xacro (robot description, xacro)
@@ -1,30 +1,30 @@
 <?xml version="1.0"?>
 <robot xmlns:xacro="http://www.ros.org/wiki/xacro">
-    <xacro:macro name="livox_mid360" params="name parent *origin">
-        <joint name="${name}_joint" type="fixed">
-            <parent link="${parent}" />
-            <child link="${name}" />
-            <xacro:insert_block name="origin" />
-        </joint>
-        <link name="${name}">
-            <visual>
-                <geometry>
-                    <mesh filename="package://sfg_peripherals_description/mesh/livox_mid360.dae"
-                        scale="1 1 1" />
-                </geometry>
-            </visual>
-        </link>
-        <joint name="${name}_point_cloud_frame_joint" type="fixed">
-            <parent link="${name}" />
-            <child link="${name}_point_cloud_frame" />
-            <origin rpy="0 0 ${pi}" xyz="0 0 0.047" />
-        </joint>
-        <link name="${name}_point_cloud_frame" />
-        <joint name="${name}_imu_frame_joint" type="fixed">
-            <parent link="${name}" />
-            <child link="${name}_imu_frame" />
-            <origin rpy="0 0 ${pi}" xyz="-0.02329 -0.011 0.00288" />
-        </joint>
-        <link name="${name}_imu_frame" />
-    </xacro:macro>
+  <xacro:macro name="livox_mid360" params="name parent *origin">
+    <joint name="${name}_joint" type="fixed">
+      <parent link="${parent}" />
+      <child link="${name}" />
+      <xacro:insert_block name="origin" />
+    </joint>
+    <link name="${name}">
+      <visual>
+        <geometry>
+          <mesh filename="package://sfg_peripherals_description/mesh/livox_mid360.dae"
+            scale="1 1 1" />
+        </geometry>
+      </visual>
+    </link>
+    <joint name="${name}_point_cloud_frame_joint" type="fixed">
+      <parent link="${name}" />
+      <child link="${name}_point_cloud_frame" />
+      <origin rpy="0 0 ${pi}" xyz="0 0 0.047" />
+    </joint>
+    <link name="${name}_point_cloud_frame" />
+    <joint name="${name}_imu_frame_joint" type="fixed">
+      <parent link="${name}" />
+      <child link="${name}_imu_frame" />
+      <origin rpy="0 0 ${pi}" xyz="-0.02329 -0.011 0.00288" />
+    </joint>
+    <link name="${name}_imu_frame" />
+  </xacro:macro>
 </robot>

File: sfg_peripherals_description/xacro/luxonis_oakd_pro.xacro (robot description, xacro)
@@ -1,64 +1,64 @@
 <?xml version="1.0"?>
 <robot xmlns:xacro="http://www.ros.org/wiki/xacro">
-    <xacro:macro name="luxonis_oakd_pro" params="name parent *origin">
-        <joint name="${name}_joint" type="fixed">
-            <parent link="${parent}" />
-            <child link="${name}" />
-            <xacro:insert_block name="origin" />
-        </joint>
-        <link name="${name}">
-            <visual>
-                <geometry>
-                    <mesh
-                        filename="package://sfg_peripherals_description/mesh/luxonis_oakd_pro.dae"
-                        scale="1 1 1" />
-                </geometry>
-            </visual>
-        </link>
-        <joint name="${name}_base_frame_joint" type="fixed">
-            <parent link="${name}" />
-            <child link="${name}_base_frame" />
-            <origin rpy="0 ${-0.5 * pi} 0" xyz="0 0.00476 0.02273" />
-        </joint>
-        <link name="${name}_base_frame" />
-        <!-- color -->
-        <joint name="${name}_color_frame_joint" type="fixed">
-            <parent link="${name}_base_frame" />
-            <child link="${name}_color_frame" />
-            <origin rpy="0 0 0" xyz="0 0 0" />
-        </joint>
-        <link name="${name}_color_frame" />
-        <joint name="${name}_color_optical_frame_joint" type="fixed">
-            <parent link="${name}_color_frame" />
-            <child link="${name}_color_optical_frame" />
-            <origin rpy="${-0.5 * pi} 0 ${-0.5 * pi}" xyz="0 0 0" />
-        </joint>
-        <link name="${name}_color_optical_frame" />
-        <!-- mono left -->
-        <joint name="${name}_mono_left_frame_joint" type="fixed">
-            <parent link="${name}_base_frame" />
-            <child link="${name}_mono_left_frame" />
-            <origin rpy="0 0 0" xyz="0 0.0375 0" />
-        </joint>
-        <link name="${name}_mono_left_frame" />
-        <joint name="${name}_mono_left_optical_frame_joint" type="fixed">
-            <parent link="${name}_mono_left_frame" />
-            <child link="${name}_mono_left_optical_frame" />
-            <origin rpy="${-0.5 * pi} 0 ${-0.5 * pi}" xyz="0 0 0" />
-        </joint>
-        <link name="${name}_mono_left_optical_frame" />
-        <!-- mono right -->
-        <joint name="${name}_mono_right_frame_joint" type="fixed">
-            <parent link="${name}_base_frame" />
-            <child link="${name}_mono_right_frame" />
-            <origin rpy="0 0 0" xyz="0 -0.0375 0" />
-        </joint>
-        <link name="${name}_mono_right_frame" />
-        <joint name="${name}_mono_right_optical_frame_joint" type="fixed">
-            <parent link="${name}_mono_right_frame" />
-            <child link="${name}_mono_right_optical_frame" />
-            <origin rpy="${-0.5 * pi} 0 ${-0.5 * pi}" xyz="0 0 0" />
-        </joint>
-        <link name="${name}_mono_right_optical_frame" />
-    </xacro:macro>
+  <xacro:macro name="luxonis_oakd_pro" params="name parent *origin">
+    <joint name="${name}_joint" type="fixed">
+      <parent link="${parent}" />
+      <child link="${name}" />
+      <xacro:insert_block name="origin" />
+    </joint>
+    <link name="${name}">
+      <visual>
+        <geometry>
+          <mesh
+            filename="package://sfg_peripherals_description/mesh/luxonis_oakd_pro.dae"
+            scale="1 1 1" />
+        </geometry>
+      </visual>
+    </link>
+    <joint name="${name}_base_frame_joint" type="fixed">
+      <parent link="${name}" />
+      <child link="${name}_base_frame" />
+      <origin rpy="0 ${-0.5 * pi} 0" xyz="0 0.00476 0.02273" />
+    </joint>
+    <link name="${name}_base_frame" />
+    <!-- color -->
+    <joint name="${name}_color_frame_joint" type="fixed">
+      <parent link="${name}_base_frame" />
+      <child link="${name}_color_frame" />
+      <origin rpy="0 0 0" xyz="0 0 0" />
+    </joint>
+    <link name="${name}_color_frame" />
+    <joint name="${name}_color_optical_frame_joint" type="fixed">
+      <parent link="${name}_color_frame" />
+      <child link="${name}_color_optical_frame" />
+      <origin rpy="${-0.5 * pi} 0 ${-0.5 * pi}" xyz="0 0 0" />
+    </joint>
+    <link name="${name}_color_optical_frame" />
+    <!-- mono left -->
+    <joint name="${name}_mono_left_frame_joint" type="fixed">
+      <parent link="${name}_base_frame" />
+      <child link="${name}_mono_left_frame" />
+      <origin rpy="0 0 0" xyz="0 0.0375 0" />
+    </joint>
+    <link name="${name}_mono_left_frame" />
+    <joint name="${name}_mono_left_optical_frame_joint" type="fixed">
+      <parent link="${name}_mono_left_frame" />
+      <child link="${name}_mono_left_optical_frame" />
+      <origin rpy="${-0.5 * pi} 0 ${-0.5 * pi}" xyz="0 0 0" />
+    </joint>
+    <link name="${name}_mono_left_optical_frame" />
+    <!-- mono right -->
+    <joint name="${name}_mono_right_frame_joint" type="fixed">
+      <parent link="${name}_base_frame" />
+      <child link="${name}_mono_right_frame" />
+      <origin rpy="0 0 0" xyz="0 -0.0375 0" />
+    </joint>
+    <link name="${name}_mono_right_frame" />
+    <joint name="${name}_mono_right_optical_frame_joint" type="fixed">
+      <parent link="${name}_mono_right_frame" />
+      <child link="${name}_mono_right_optical_frame" />
+      <origin rpy="${-0.5 * pi} 0 ${-0.5 * pi}" xyz="0 0 0" />
+    </joint>
+    <link name="${name}_mono_right_optical_frame" />
+  </xacro:macro>
 </robot>
