Commit message: Updated Collision and Inertia for Intel RealSense D435.

File: sfg_peripherals_description/xacro/intel_realsense_d435.xacro (robot description, xacro)
@@ -11,8 +11,19 @@
         <geometry>
           <mesh
-            filename="package://sfg_peripherals_description/mesh/intel_realsense_d435.dae"
-            scale="1 1 1" />
+            filename="package://sfg_peripherals_description/mesh/intel_realsense_d435.dae" />
         </geometry>
       </visual>
+      <collision>
+        <geometry>
+          <mesh
+            filename="package://sfg_peripherals_description/mesh/intel_realsense_d435.dae" />
+        </geometry>
+      </collision>
+      <inertial>
+        <origin xyz="0.001113 -0.0000279 0.012428" rpy="0 0 ${-pi/2}" />
+        <mass value="0.072" />
+        <inertia ixx="0.000017639" ixy="0" ixz="-0.00000035" iyy="0.000055074"
+          iyz="0.000000037" izz="0.000043502" />
+      </inertial>
     </link>
     <joint name="${name}_base_frame_joint" type="fixed">

Commit message: sfg_peripherals_description: change realsense base frame to optical color frame.

File: sfg_peripherals_description/xacro/intel_realsense_d435.xacro (robot description, xacro)
@@ -27,10 +27,10 @@
       </inertial>
     </link>
-    <joint name="${name}_base_frame_joint" type="fixed">
+    <joint name="${name}_color_optical_frame_joint" type="fixed">
       <parent link="${name}" />
-      <child link="${name}_base_frame" />
-      <origin rpy="0 ${-0.5 * pi} 0" xyz="0 0.0175 0.02075" />
+      <child link="${name}_color_optical_frame" />
+      <origin rpy="0 ${-0.5 * pi} 0" xyz="0 0.0325 0.02085" />
     </joint>
-    <link name="${name}_base_frame" />
+    <link name="${name}_color_optical_frame" />
   </xacro:macro>
 </robot>

Commit message: sfg_peripherals_description: Distinguise between color and color optical frame.

File: sfg_peripherals_description/xacro/intel_realsense_d435.xacro (robot description, xacro)
@@ -27,8 +27,14 @@
       </inertial>
     </link>
+    <joint name="${name}_color_frame_joint" type="fixed">
+      <parent link="${name}" />
+      <child link="${name}_color_frame" />
+      <origin rpy="0 ${-0.5 * pi} 0" xyz="0 0.0325 0.02085" />
+    </joint>
+    <link name="${name}_color_frame" />
     <joint name="${name}_color_optical_frame_joint" type="fixed">
       <parent link="${name}" />
       <child link="${name}_color_optical_frame" />
-      <origin rpy="0 ${-0.5 * pi} 0" xyz="0 0.0325 0.02085" />
+      <origin rpy="0 0 ${-0.5 * pi}" xyz="0 0.0325 0.02085" />
     </joint>
     <link name="${name}_color_optical_frame" />
