Commit message: sfg_peripherals_description: Removed htc_vive_tracker_30 and added base_marker_tree.

File: sfg_peripherals_description/xacro/base_marker_tree.xacro (robot description, xacro)
@@ -1,5 +1,5 @@
 <?xml version="1.0"?>
 <robot xmlns:xacro="http://www.ros.org/wiki/xacro">
-  <xacro:macro name="htc_vive_tracker_30" params="name parent *origin">
+  <xacro:macro name="base_marker_tree" params="name parent *origin">
     <joint name="${name}_joint" type="fixed">
       <parent link="${parent}" />
@@ -11,5 +11,5 @@
         <geometry>
           <mesh
-            filename="package://sfg_peripherals_description/mesh/htc_vive_tracker_30.dae"
+            filename="package://sfg_peripherals_description/mesh/base_marker_tree.dae"
             scale="1 1 1" />
         </geometry>
@@ -19,5 +19,5 @@
       <parent link="${name}" />
       <child link="${name}_frame" />
-      <origin rpy="${0.5 * pi} 0 ${-0.5 * pi}" xyz="0 0 0.0005" />
+      <origin rpy="0 0 0" xyz="0 0 0" />
     </joint>
     <link name="${name}_frame" />

Commit message: sfg_peripherals_description: Switched from .dae to .glb files.

File: sfg_peripherals_description/xacro/base_marker_tree.xacro (robot description, xacro)
@@ -9,8 +9,8 @@
     <link name="${name}">
       <visual>
+        <origin xyz="0 0 0" rpy="${0.5 * pi} 0 ${0.5 * pi}" />
         <geometry>
           <mesh
-            filename="package://sfg_peripherals_description/mesh/base_marker_tree.dae"
-            scale="1 1 1" />
+            filename="package://sfg_peripherals_description/mesh/base_marker_tree.glb" scale="1 1 1" />
         </geometry>
       </visual>

File: sfg_peripherals_description/xacro/intel_realsense_d435.xacro (robot description, xacro)
@@ -9,21 +9,11 @@
     <link name="${name}">
       <visual>
+        <origin xyz="0 0 0" rpy="${0.5 * pi} 0 ${0.5 * pi}" />
         <geometry>
           <mesh
-            filename="package://sfg_peripherals_description/mesh/intel_realsense_d435.dae" />
+            filename="package://sfg_peripherals_description/mesh/intel_realsense_d435.glb"
+            scale="1 1 1" />
         </geometry>
       </visual>
-      <collision>
-        <geometry>
-          <mesh
-            filename="package://sfg_peripherals_description/mesh/intel_realsense_d435.dae" />
-        </geometry>
-      </collision>
-      <inertial>
-        <origin xyz="0.001113 -0.0000279 0.012428" rpy="0 0 ${-pi/2}" />
-        <mass value="0.072" />
-        <inertia ixx="0.000017639" ixy="0" ixz="-0.00000035" iyy="0.000055074"
-          iyz="0.000000037" izz="0.000043502" />
-      </inertial>
     </link>
     <joint name="${name}_color_frame_joint" type="fixed">

File: sfg_peripherals_description/xacro/livox_mid360.xacro (robot description, xacro)
@@ -9,7 +9,7 @@
     <link name="${name}">
       <visual>
+        <origin xyz="0 0 0" rpy="${0.5 * pi} 0 ${-0.5 * pi}" />
         <geometry>
-          <mesh filename="package://sfg_peripherals_description/mesh/livox_mid360.dae"
-            scale="1 1 1" />
+          <mesh filename="package://sfg_peripherals_description/mesh/livox_mid360.glb" scale="1 1 1" />
         </geometry>
       </visual>
@@ -24,5 +24,5 @@
       <parent link="${name}" />
       <child link="${name}_imu_frame" />
-      <origin rpy="0 0 ${pi}" xyz="-0.02329 -0.011 0.00288" />
+      <origin rpy="0 0 ${pi}" xyz="-0.011 -0.02329 0.00288" />
     </joint>
     <link name="${name}_imu_frame" />

File: sfg_peripherals_description/xacro/luxonis_oakd_pro.xacro (robot description, xacro)
@@ -9,8 +9,8 @@
     <link name="${name}">
       <visual>
+        <origin xyz="0 0 0" rpy="${0.5 * pi} 0 ${0.5 * pi}" />
         <geometry>
           <mesh
-            filename="package://sfg_peripherals_description/mesh/luxonis_oakd_pro.dae"
-            scale="1 1 1" />
+            filename="package://sfg_peripherals_description/mesh/luxonis_oakd_pro.glb" scale="1 1 1" />
         </geometry>
       </visual>

Commit message: sfg_peripherals_description: Removed default scale from .xacro files.

File: sfg_peripherals_description/xacro/base_marker_tree.xacro (robot description, xacro)
@@ -12,5 +12,5 @@
         <geometry>
           <mesh
-            filename="package://sfg_peripherals_description/mesh/base_marker_tree.glb" scale="1 1 1" />
+            filename="package://sfg_peripherals_description/mesh/base_marker_tree.glb" />
         </geometry>
       </visual>

File: sfg_peripherals_description/xacro/intel_realsense_d435.xacro (robot description, xacro)
@@ -12,6 +12,5 @@
         <geometry>
           <mesh
-            filename="package://sfg_peripherals_description/mesh/intel_realsense_d435.glb"
-            scale="1 1 1" />
+            filename="package://sfg_peripherals_description/mesh/intel_realsense_d435.glb" />
         </geometry>
       </visual>

File: sfg_peripherals_description/xacro/livox_mid360.xacro (robot description, xacro)
@@ -11,5 +11,5 @@
         <origin xyz="0 0 0" rpy="${0.5 * pi} 0 ${-0.5 * pi}" />
         <geometry>
-          <mesh filename="package://sfg_peripherals_description/mesh/livox_mid360.glb" scale="1 1 1" />
+          <mesh filename="package://sfg_peripherals_description/mesh/livox_mid360.glb" />
         </geometry>
       </visual>

File: sfg_peripherals_description/xacro/luxonis_oakd_pro.xacro (robot description, xacro)
@@ -12,5 +12,5 @@
         <geometry>
           <mesh
-            filename="package://sfg_peripherals_description/mesh/luxonis_oakd_pro.glb" scale="1 1 1" />
+            filename="package://sfg_peripherals_description/mesh/luxonis_oakd_pro.glb" />
         </geometry>
       </visual>
